Commit message: Plotting position and velocity after simulation concludes.

File: urdf/single_pendulum.urdf (robot description, URDF)
Before this commit: robot single_pendulum, 3 links, 2 joints
Joints:
- joint base_branch_joint: origin xyz=0 0 0 rpy=0 3.14159265358979323846 0 -> xyz=0 0 0 rpy=0 0 0

Commit message: Confirmed that code works with single or triple pendulum.

File: urdf/single_pendulum.urdf (robot description, URDF)
Before this commit: robot single_pendulum, 3 links, 2 joints
Joints:
- joint world_to_base: origin xyz=0 0 1.5 rpy=0 0 0 -> xyz=0 -.5 .025 rpy=0 0 0
