Commit message: triple pendulum now a reasonable height

File: urdf/typed_pends/triple_pendulum.urdf (robot description, URDF)
Before this commit: robot single_pendulum, 5 links, 4 joints
Links:
- link branch_link_a: geometry collision cylinder length=0.4 radius=0.00608; visual cylinder length=0.4 radius=0.00608
- link branch_link_b: geometry collision cylinder length=0.4 radius=0.00608; visual cylinder length=0.4 radius=0.00608
- link branch_link_c: geometry collision cylinder length=0.4 radius=0.00608; visual cylinder length=0.4 radius=0.00608
Joints:
- joint branch_joint_ab: origin xyz=0 0 0.79 rpy=0 0 0 -> xyz=0 0 0.4 rpy=0 0 0
- joint branch_joint_bc: origin xyz=0 0 0.79 rpy=0 0 0 -> xyz=0 0 0.4 rpy=0 0 0
