Commit message: Added fork to probe to capture branch in case of future 3D pendulum

File: urdf/probes/forked_probe.urdf (robot description, URDF)
Before this commit: robot forked_probe, 4 links, 3 joints
Links:
- added link crossbar_link, mass 0.005; collision cylinder length=0.035 radius=0.005; visual cylinder length=0.035 radius=0.005
- added link left_fork, mass 0.005; collision cylinder length=0.05 radius=0.005; visual cylinder length=0.05 radius=0.005
- added link right_fork, mass 0.005; collision cylinder length=0.05 radius=0.005; visual cylinder length=0.05 radius=0.005
Joints:
- added joint joint_crossbar_hilt: type fixed, parent probe_link, child crossbar_link, origin xyz=0.0975 0 0 rpy=0 0 0, axis 0 0 1, limit effort=0 velocity=0
- added joint left_fork_joint: type fixed, parent crossbar_link, child left_fork, origin xyz=0.025 0.0175 0 rpy=0 0 0, axis 0 0 1, limit effort=0 velocity=0
- added joint right_fork_joint: type fixed, parent crossbar_link, child right_fork, origin xyz=0.025 -0.0175 0 rpy=0 0 0, axis 0 0 1, limit effort=0 velocity=0

Commit message: plots joint angles and probe values after finishing a run

File: urdf/probes/forked_probe.urdf (robot description, URDF)
Before this commit: robot forked_probe, 7 links, 6 joints
Joints:
- joint base_joint: origin xyz=0 0 0 rpy=0 0 0 -> xyz=-.005 0 0 rpy=0 0 0
- joint joint_sensor: origin xyz=0.1 0 0 rpy=0 0 0 -> xyz=.1 0 0 rpy=0 0 0

Commit message: use contact normal instead of f/t sensor to measure forces

File: urdf/probes/forked_probe.urdf (robot description, URDF)
Before this commit: robot forked_probe, 7 links, 6 joints
Links:
- link sensor_link: geometry collision box size=.02 .02 .02; visual box size=.02 .02 .02
